File: RibbonCable_MB_BreakdownBoard/RibbonCable_MB_BreakdownBoard.kicad_pcb (KiCad board)
At the start: 2 copper layers, 60 x 35 mm, 24 parts, among them J1 EEPROM I2C, U1 AT24C256

Commit message: updated silkscreen to have more info
Parts:
- renumbered X_FAN1 to E/K_FAN1
Routing:
- net Net-(FAN1-Pad2): track 12.0 -> 23.9 mm
- net Net-(FIL_SENS1-Pad1): track 58.5 -> 69.2 mm
- net Net-(Ribbon1-Pad11): track 27.1 -> 30.8 mm
Other:
- board text added: "+ve"
- board text added: "CR-10S Pro ribbon cable MB breakdown board With EEPROM V1.1a 19/10/2019"
- board text added: "GND"
- board text removed: "CR-10S Pro ribbon cable MB breakdown board With EEPROM V1.1 14/10/2019"
