File: RibbonCable_MB_BreakdownBoard/RibbonCable_MB_BreakdownBoard.sch (KiCad schematic (older format))
At the start: 19 parts, among them J1 EEPROM I2C, U1 AT24C256

Commit message: updated silkscreen to have more info
Parts:
- renumbered X_FAN1 to E/K_FAN1
Changed lines of the file:
@@
 $EndComp
 $Comp
-L Connector_Generic:Conn_01x02 X_FAN1
+L Connector_Generic:Conn_01x02 E/K_FAN1
 U 1 1 5D528B45
 P 7500 2150
-F 0 "X_FAN1" H 7580 2142 50  0000 L CNN
+F 0 "E/K_FAN1" H 7580 2142 50  0000 L CNN
 F 1 "Conn_01x02" H 7580 2051 50  0000 L CNN
 F 2 "Connector_JST:JST_XH_B2B-XH-A_1x02_P2.50mm_Vertical" H 7580 2005 50  0001 L CNN
